File: ADC/ADC.kicad_sch (KiCad schematic)
At the start: 77 parts, among them IC1 ADS7953SDBT, IC2 REF5025ID, IC3 ADS7953SDBT, IC4 REF5025ID, IC5 ADP3338AKCZ-5-REEL, J1 USB_C_Receptacle_USB2.0, J2 Conn_01x04_MountingPin, J3 Conn_02x11_Odd_Even, J4 Conn_02x08_Top_Bottom, J5 Conn_02x08_Top_Bottom, J6 Conn_01x04_MountingPin, J7 Conn_02x05_Odd_Even, U1 STM32F072CBT6, U2 OPA192ID, U3 PRTR5V0U2X, U4 XC6206PxxxMR-Regulator_Linear, U5 OPA192ID

Commit message: updated schematic to match the eval kit
Parts:
- removed J3: Conn_02x11_Odd_Even, Connector_PinHeader_2.54mm:PinHeader_2x11_P2.54mm_Vertical, symbol Connector_Generic:Conn_02x11_Odd_Even
- removed J4, J5: Conn_02x08_Top_Bottom, Connector_PinHeader_2.54mm:PinHeader_2x08_P2.54mm_Vertical, symbol Connector_Generic:Conn_02x08_Counter_Clockwise
- removed J7: Conn_02x05_Odd_Even, Connector_PinHeader_2.54mm:PinHeader_2x05_P2.54mm_Vertical, symbol Connector_Generic:Conn_02x05_Odd_Even
- removed SW1: ~, Button_Switch_SMD:SW_Push_SPST_NO_Alps_SKRK, symbol Switch:SW_Push
- added AC1: LSM6DSOTR, SamacSys_Parts:LGA-14_2.5X3X0.86_, symbol SamacSys_Parts:LSM6DSOTR
- added C53, C54, C55, C57, C58, C61, C62: 100nF, Capacitor_SMD:C_0402_1005Metric, symbol Device:C
- added C56: 220nF, Capacitor_SMD:C_0402_1005Metric, symbol Device:C
- added C59, C60: 1uF, Capacitor_SMD:C_0402_1005Metric, symbol Device:C
- added C63: 10µF, Capacitor_SMD:C_0402_1005Metric, symbol Device:C
- added H1, H2, H3, H4: MountingHole_Pad, MountingHole:MountingHole_3mm_Pad, symbol Mechanical:MountingHole_Pad
- added J10, J11, J12, J13, J14, J8, J9: Conn_01x04_MountingPin, Connector_JST:JST_PH_B4B-PH-K_1x04_P2.00mm_Vertical, symbol Connector_Generic:Conn_01x04
- added J15, J16, J4, J5: Conn_01x02, Connector_Molex:Molex_PicoBlade_53047-0210_1x02_P1.25mm_Vertical, symbol Connector_Generic:Conn_01x02
- added R10, R11, R12, R13, R14, R15, R16, R17, R18, R19, R20, R21, R22, R23, R24, R25, R26, R27, R28, R29, R30, R31, R32, R33, R34, R35, R36, R37, R38, R39, R40, R41, R8, R9: 33, symbol Device:R_US
- added R6, R7: 10k, Resistor_SMD:R_0603_1608Metric_Pad0.98x0.95mm_HandSolder, symbol Device:R_Small_US
- added S1, S2: SKQGABE010, SKQGAKE010, symbol SamacSys_Parts:SKQGABE010
- added SW1: SW_SPDT, symbol Switch:SW_SPDT
- added TP1, TP10, TP11, TP12, TP2, TP3, TP4, TP5, TP6, TP7, TP8, TP9: TestPoint, symbol Connector:TestPoint
- added U6: SHT4x, Sensor_Humidity:Sensirion_DFN-4_1.5x1.5mm_P0.8mm_SHT4x_NoCentralPad, symbol Sensor_Humidity:SHT4x
- added U7: LIS3MDL, Package_LGA:LGA-12_2x2mm_P0.5mm, symbol Sensor_Magnetic:LIS3MDL
- C1, C2: value 1µF -> 100nF; footprint Capacitor_SMD:C_0201_0603Metric -> Capacitor_SMD:C_0402_1005Metric
- C10, C11, C12, C3, C33, C4, C42, C5, C6, C7, C8: footprint Capacitor_SMD:C_0201_0603Metric -> Capacitor_SMD:C_0402_1005Metric
- C13, C14, C15, C16, C17, C18, C19, C20, C21, C22, C23, C24, C25, C26, C27, C28, C29, C30, C31, C32, C34, C35, C36, C37, C38, C39, C40, C41, C43, C44, C45, C46, C47, C48: value 150pF -> 270pF; footprint Capacitor_SMD:C_0201_0603Metric -> Capacitor_SMD:C_0402_1005Metric
- C50, C51: value 1µF -> 10uF; footprint Capacitor_SMD:C_0201_0603Metric -> Capacitor_SMD:C_0402_1005Metric
- C52: value 10µF -> 100nF
- R2, R3: symbol Device:R -> Device:R_US
- R4, R5: value 100 -> 33
Connections:
- net +3.3V: now also AC1.1 (SDO/SA0), AC1.12 (CS), AC1.5 (VDDIO), AC1.8 (VDD), C53.2, C54.2, C56.2, C57.2, C58.2, C61.2, C62.2, R6.1, R7.1, S1.1, S1.3, S2.2, S2.4, TP9.1, U6.3 (VDD), U7.10 (~{CS}), U7.5 (Vdd), U7.6 (Vdd_IO), U7.9 (SDO/SA1); no longer J2.2 (Pin_2)
- net +5V: now also C59.1, C60.1, J15.1 (Pin_1), J16.1 (Pin_1), J4.1 (Pin_1), J5.1 (Pin_1), TP10.1
- net A0: now also R8.1
- net A1: now also R9.1
- net A10: now also R18.1
- net A11: now also R19.1
- net A12: now also R20.1
- net A13: now also R21.1
- net A14: now also R22.1
- net A15: now also R23.1
- net A16: now also R24.2
- net A17: now also R25.2
- net A18: now also R26.2
- net A19: now also R27.2
- net A2: now also R10.1
- net A20: now also R28.2
- net A21: now also R29.2
- net A22: now also R30.2
- net A23: now also R31.2
- net A24: now also R32.2
- net A25: now also R33.2
- net A26: now also R34.2
- net A27: now also R35.2
- net A28: now also R36.2
- net A29: now also R37.2
- net A3: now also R11.1
- net A30: now also R38.2
- net A31: now also R39.2
- net A4: now also R12.1
- net A5: now also R13.1
- net A6: now also R14.1
- net A7: now also R15.1
- net A8: now also R16.1
- net A9: now also R17.1
- net BOOT0: now also S1.2, S1.4
- net CS_SPI: now also TP4.1, TP8.1
- net GND: now also AC1.6 (GND_1), AC1.7 (GND_2), C53.1, C54.1, C55.1, C56.1, C57.1, C58.1, C59.2, C60.2, C61.1, C62.1, C63.1, H1.1, H2.1, H3.1, H4.1, J15.2 (Pin_2), J16.2 (Pin_2), J4.2 (Pin_2), J5.2 (Pin_2), U6.4 (VSS), U7.12 (GND), U7.2 (GND), U7.3 (GND); no longer J2.1 (Pin_1)
- net MISO_SPI1: now also R40.2, TP1.1; no longer IC1.34 (SDO)
- net MISO_SPI2: now also R41.2, TP5.1; no longer IC3.34 (SDO)
- net MOSI_SPI1: now also TP2.1
- net MOSI_SPI2: now also TP6.1
- net NRST: now also S2.1, S2.3
- net REFIN1: now also C55.2
- net REFIN2: now also C63.2
- net SCK_SPI1: now also TP3.1
- net SCK_SPI2: now also TP7.1
- net SCL_I2C1: now also AC1.13 (SCL), R7.2, U6.2 (SCL), U7.1 (SCL/SPC); no longer J2.3 (Pin_3)
- net SDA_I2C1: now also AC1.14 (SDA), R6.2, U6.1 (SDA), U7.11 (SDA/SDI/SDO); no longer J2.4 (Pin_4)
- net VBUS: now also SW1.2 (B); no longer F1.1, J1.A4 (VBUS), J1.A9 (VBUS), J1.B4 (VBUS), J1.B9 (VBUS)
- removed net POWER: IC1.2 (GPIO3), IC3.2 (GPIO3), U1.38 (PA15)
- removed net RANGE_SEL: IC1.1 (GPIO2), IC3.1 (GPIO2), U1.25 (PB12)
- new net: J14.2 (Pin_2), R37.1
- new net: J12.2 (Pin_2), R25.1
- new net: J10.4 (Pin_4), R23.2
- new net: J13.2 (Pin_2), R33.1
- new net: J11.1 (Pin_1), R28.1
- new net: J11.2 (Pin_2), R29.1
- new net: J11.3 (Pin_3), R30.1
- new net: J11.4 (Pin_4), R31.1
- new net: J10.3 (Pin_3), R22.2
- new net: J8.4 (Pin_4), R15.2
- new net: J12.1 (Pin_1), R24.1
- new net: J13.3 (Pin_3), R34.1
- new net: J9.1 (Pin_1), R16.2
- new net: J2.4 (Pin_4), R11.2
- new net: J12.4 (Pin_4), R27.1
- new net: J12.3 (Pin_3), R26.1
- new net: J8.2 (Pin_2), R13.2
- new net: J1.A4 (VBUS), J1.A9 (VBUS), J1.B4 (VBUS), J1.B9 (VBUS)
- new net: IC1.34 (SDO), R40.1
- new net: J2.1 (Pin_1), R8.2
- new net: J2.2 (Pin_2), R9.2
- new net: J2.3 (Pin_3), R10.2
- new net: SW1.1 (A), TP11.1
- new net: J13.4 (Pin_4), R35.1
- new net: IC3.34 (SDO), R41.1
- new net: J13.1 (Pin_1), R32.1
- new net: J14.4 (Pin_4), R39.1
- new net: J8.1 (Pin_1), R12.2
- new net: J8.3 (Pin_3), R14.2
- new net: J9.2 (Pin_2), R17.2
- new net: J9.3 (Pin_3), R18.2
- new net: J9.4 (Pin_4), R19.2
- new net: J14.1 (Pin_1), R36.1
- new net: J10.1 (Pin_1), R20.2
- new net: J10.2 (Pin_2), R21.2
- new net: J14.3 (Pin_3), R38.1
- new net PA15: U1.38 (PA15)
- new net PB12: U1.25 (PB12)
- new net VBUS_IN: F1.1, SW1.3 (C), TP12.1
- no-connect marks 20 -> 33
Other:
- note removed: "EXTRA GPIO"
- note removed: "I2C CONNECTOR FOR O2 SENSOR"
- note removed: "POWER, GROUND AND MORE GROUND"
- moved on the sheet: C10, C11, C12, C13, C49, C5, F1, IC2, IC4, IC5, J6, R1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

Commit message: finished V2
Parts:
- removed TP1, TP2, TP3, TP5, TP6, TP7, TP8: TestPoint, symbol Connector:TestPoint
- R1, R2, R3, R4, R5, R6, R7: footprint Resistor_SMD:R_0603_1608Metric_Pad0.98x0.95mm_HandSolder -> Resistor_SMD:R_0402_1005Metric_Pad0.72x0.64mm_HandSolder
- R10, R11, R12, R13, R14, R15, R16, R17, R18, R19, R20, R21, R22, R23, R24, R25, R26, R27, R28, R29, R30, R31, R32, R33, R34, R35, R36, R37, R38, R39, R40, R41, R8, R9: footprint (none) -> Resistor_SMD:R_0402_1005Metric_Pad0.72x0.64mm_HandSolder
- SW1: footprint (none) -> Button_Switch_SMD:SW_SPDT_CK_JS102011SAQN
- TP10, TP11, TP12, TP4, TP9: footprint (none) -> TestPoint:TestPoint_Pad_D1.0mm
Connections:
- net +5V: now also J15.2 (Pin_2), J16.2 (Pin_2), J4.2 (Pin_2), J5.2 (Pin_2); no longer J15.1 (Pin_1), J16.1 (Pin_1), J4.1 (Pin_1), J5.1 (Pin_1)
- net GND: now also J15.1 (Pin_1), J16.1 (Pin_1), J4.1 (Pin_1), J5.1 (Pin_1); no longer J15.2 (Pin_2), J16.2 (Pin_2), J4.2 (Pin_2), J5.2 (Pin_2)
- net VBUS: now also J1.A4 (VBUS), J1.A9 (VBUS), J1.B4 (VBUS), J1.B9 (VBUS)
- net PA0: no longer names the net of U1.10 (PA0)
- net PA1: no longer names the net of U1.11 (PA1)
- net PA10: no longer names the net of U1.31 (PA10)
- net PA13: no longer names the net of U1.34 (PA13)
- net PA14: no longer names the net of U1.37 (PA14)
- net PA15: no longer names the net of U1.38 (PA15)
- net PA2: no longer names the net of U1.12 (PA2)
- net PA3: no longer names the net of U1.13 (PA3)
- net PA8: no longer names the net of U1.29 (PA8)
- net PA9: no longer names the net of U1.30 (PA9)
- net PB0: no longer names the net of U1.18 (PB0)
- net PB1: no longer names the net of U1.19 (PB1)
- net PB12: no longer names the net of U1.25 (PB12)
- net PB2: no longer names the net of U1.20 (PB2)
- net PB3: no longer names the net of U1.39 (PB3)
- net PB4: no longer names the net of U1.40 (PB4)
- net PB5: no longer names the net of U1.41 (PB5)
- net PB8: no longer names the net of U1.45 (PB8)
- net PB9: no longer names the net of U1.46 (PB9)
- net PC13: no longer names the net of U1.2 (PC13)
- net PC14: no longer names the net of U1.3 (PC14)
- net PC15: no longer names the net of U1.4 (PC15)
- net PF0: no longer names the net of U1.5 (PF0)
- net PF1: no longer names the net of U1.6 (PF1)
- no-connect marks 33 -> 57

Commit message: updated v2
Parts:
- removed TP4: TestPoint, TestPoint:TestPoint_Pad_D1.0mm, symbol Connector:TestPoint

Commit message: updated code
Parts:
- C11, C12, C33, C42: value 1µF -> 1uF
- C49, C63, C9: value 10µF -> 10uF
Changed lines of the file:
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@@
 			)
 		)
-		(property "Value" "1µF"
+		(property "Value" "1uF"
 			(at 229.87 147.3199 0)
 			(effects
@@
 			)
 		)
-		(property "Value" "1µF"
+		(property "Value" "1uF"
 			(at 259.08 41.275 0)
 			(effects
@@
 			)
 		)
-		(property "Value" "1µF"
+		(property "Value" "1uF"
 			(at 281.94 41.275 0)
 			(effects
@@
 			)
 		)
-		(property "Value" "10µF"
+		(property "Value" "10uF"
 			(at 145.161 26.543 0)
 			(effects
@@
 			)
 		)
-		(property "Value" "10µF"
+		(property "Value" "10uF"
 			(at 76.2 135.8899 0)
 			(effects
@@
 			)
 		)
-		(property "Value" "1µF"
+		(property "Value" "1uF"
 			(at 331.47 140.9699 0)
 			(effects
@@
 			)
 		)
-		(property "Value" "10µF"
+		(property "Value" "10uF"
 			(at 251.46 135.8899 0)
 			(effects

Commit message: pcb update
Parts:
- removed S1, S2: SKQGABE010, SKQGAKE010, symbol SamacSys_Parts:SKQGABE010
- added SW2, SW3: SW_Push, Button_Switch_SMD:SW_Push_SPST_NO_Alps_SKRK, symbol Switch:SW_Push
- U4: value XC6206PxxxMR-Regulator_Linear -> XC6206P332PR-G
Connections:
- net +3.3V: now also SW2.1, SW3.1
- net BOOT0: now also SW3.2
- net NRST: now also SW2.2

Commit message: finished v2
Parts:
- removed AC1: LSM6DSOTR, SamacSys_Parts:LGA-14_2.5X3X0.86_, symbol SamacSys_Parts:LSM6DSOTR
- removed C13, C14, C15, C16, C17, C19, C20, C21, C23, C24, C27, C36, C38, C39, C40, C41, C43, C44, C45, C46, C47, C48: 270pF, Capacitor_SMD:C_0402_1005Metric, symbol Device:C
- removed C53, C54, C57, C58: 100nF, Capacitor_SMD:C_0402_1005Metric, symbol Device:C
- removed C56: 220nF, Capacitor_SMD:C_0402_1005Metric, symbol Device:C
- removed C59, C60: 1uF, Capacitor_SMD:C_0402_1005Metric, symbol Device:C
- removed IC1, IC3: ADS7953SDBT, SOP50P640X120-38N, symbol SamacSys_Parts:ADS7953SDBT
- removed IC2, IC4: REF5025ID, SOIC127P600X175-8N, symbol SamacSys_Parts:REF5025ID
- removed IC5: ADP3338AKCZ-5-REEL, SOT230P700X180-4N, symbol SamacSys_Parts:ADP3338AKCZ-5-REEL
- removed J10, J11, J12, J13, J14, J2, J6, J8, J9: Conn_01x04_MountingPin, Connector_JST:JST_PH_B4B-PH-K_1x04_P2.00mm_Vertical, symbol Connector_Generic:Conn_01x04
- removed J15, J16, J4, J5: Conn_01x02, Connector_Molex:Molex_PicoBlade_53047-0210_1x02_P1.25mm_Vertical, symbol Connector_Generic:Conn_01x02
- removed R10, R11, R12, R13, R14, R15, R16, R17, R18, R19, R20, R21, R22, R23, R24, R25, R26, R27, R28, R29, R30, R31, R32, R33, R34, R35, R36, R37, R38, R39, R5: 33, Resistor_SMD:R_0402_1005Metric_Pad0.72x0.64mm_HandSolder, symbol Device:R_US
- removed R6, R7: 10k, Resistor_SMD:R_0402_1005Metric_Pad0.72x0.64mm_HandSolder, symbol Device:R_Small_US
- removed U2, U5: OPA192ID, SOIC127P600X175-8N, symbol SamacSys_Parts:OPA192ID
- removed U6: SHT4x, Sensor_Humidity:Sensirion_DFN-4_1.5x1.5mm_P0.8mm_SHT4x_NoCentralPad, symbol Sensor_Humidity:SHT4x
- removed U7: LIS3MDL, Package_LGA:LGA-12_2x2mm_P0.5mm, symbol Sensor_Magnetic:LIS3MDL
- added C3: 1uF, Capacitor_SMD:C_0402_1005Metric, symbol Device:C
- added C6: 100nF, Capacitor_SMD:C_0402_1005Metric, symbol Device:C
- added C9: 10uF, Capacitor_SMD:C_0402_1005Metric, symbol Device:C
- added R7: 33, Resistor_SMD:R_0402_1005Metric_Pad0.72x0.64mm_HandSolder, symbol Device:R_US
- added U11: ADP3338AKCZ-5-REEL, footprint:SOT230P700X180-4N, symbol ADP3338AKCZ-5-REEL:ADP3338AKCZ-5-REEL
- added U2, U3, U4: ADS7953SDBT, footprint:DBT38, symbol ADS7953SDBT:ADS7953SDBT
- added U5, U7, U8: OPA192ID, footprint:SOIC127P599X175-8N, symbol OPA192ID:OPA192ID
- added U9: REF5025ID, footprint:SOIC127P599X175-8N, symbol REF5025ID:REF5025ID
- C18, C26, C28, C29, C30, C31: value 270pF -> 1uF
- C22: value 270pF -> 10uF
- C25: value 270pF -> 100nF
- C27: renamed from C10; value 100nF -> 1uF
- C37: value 270pF -> 1uF; LCSC (none) -> C307331
- renumbered C3 to C10, C4 to C11, C6 to C12, C5 to C13, C7 to C14, C8 to C15, C9 to C16, C42 to C17, C2 to C19, C33 to C2, C50 to C20, C51 to C21, C61 to C23, C62 to C24, C11 to C33, C12 to C36, C55 to C4, C52 to C5, C49 to C7, C63 to C8, R40 to R2, R41 to R3, R2 to R5, R3 to R6, SW3 to SW1, SW1 to SW3, TP11 to TP1, TP12 to TP2, TP9 to TP3, TP10 to TP4, U4 to U10, U3 to U6
Connections:
- net REFIN2 is gone; now on net REFIN: C5.2, C8.2
- net SCL_I2C2 is gone; now on net SCK_SPI2: U1.26 (PB13)
- net +3.3V: no longer C1.1, C17.1, C19.1, C2.1, C20.2, C21.2, C23.2, C24.2
- net +5V: now also C1.1, C17.1, C18.1, C19.1, C2.1, C20.2, C21.2, C22.2, C23.2, C24.2, C25.2, C26.1, C28.1, C29.1, C31.1, C37.1, C3.1, U11.2 (OUT), U11.4 (OUT__1), U2.29 (+VA_2), U2.36 (+VBD), U2.5 (+VA_1), U3.29 (+VA_2), U3.36 (+VBD), U3.5 (+VA_1), U4.29 (+VA_2), U4.36 (+VBD), U4.5 (+VA_1), U5.7 (V+), U7.7 (V+), U8.7 (V+), U9.2 (VIN)
- net +AMP1: now also U2.7 (MXO), U8.3 (+IN)
- net +AMP2: now also U3.7 (MXO), U7.3 (+IN)
- net A0: now also U2.28 (CH0); no longer C28.1, R8.1
- net A1: now also U2.27 (CH1); no longer R9.1
- net A10: now also U2.16 (CH10)
- net A11: now also U2.15 (CH11); no longer C18.1
- net A12: now also U2.14 (CH12)
- net A13: now also U2.13 (CH13)
- net A14: now also U2.12 (CH14)
- net A15: now also U2.11 (CH15)
- net A16: now also U4.28 (CH0)
- net A17: now also U4.27 (CH1)
- net A18: now also U4.26 (CH2)
- net A19: now also U4.25 (CH3)
- net A2: now also U2.26 (CH2); no longer C26.1
- net A20: now also U4.24 (CH4)
- net A21: now also U4.23 (CH5)
- net A22: now also U4.22 (CH6)
- net A23: now also U4.21 (CH7); no longer C37.1
- net A24: now also U4.18 (CH8)
- net A25: now also U4.17 (CH9)
- net A26: now also U4.16 (CH10); no longer C35.1
- net A27: now also U4.15 (CH11); no longer C34.1
- net A28: now also U4.14 (CH12); no longer C32.1
- net A29: now also U4.13 (CH13); no longer C31.1
- net A3: now also U2.25 (CH3); no longer C25.1
- net A30: now also U4.12 (CH14); no longer C30.1
- net A31: now also U4.11 (CH15); no longer C29.1
- net A4: now also U2.24 (CH4)
- net A5: now also U2.23 (CH5)
- net A6: now also U2.22 (CH6); no longer C22.1
- net A7: now also U2.21 (CH7)
- net A8: now also U2.18 (CH8)
- net A9: now also U2.17 (CH9)
- net GND: now also C22.1, C25.1, C3.2, C6.1, C9.1, U11.1 (GND), U2.10 (AGND_2), U2.19 (AGND_3), U2.20 (AGND_4), U2.3 (REFM), U2.30 (AGND_5), U2.35 (BDGND), U2.6 (AGND_1), U2.9 (AINM), U3.10 (AGND_2), U3.19 (AGND_3), U3.20 (AGND_4), U3.3 (REFM), U3.30 (AGND_5), U3.35 (BDGND), U3.6 (AGND_1), U3.9 (AINM), U4.10 (AGND_2), U4.19 (AGND_3), U4.20 (AGND_4), U4.3 (REFM), U4.30 (AGND_5), U4.35 (BDGND), U4.6 (AGND_1), U4.9 (AINM), U5.4 (-V), U7.4 (-V), U8.4 (-V), U9.4 (GND); no longer C22.2, C25.2
- net MOSI_SPI1: now also U2.33 (SDI)
- net MOSI_SPI2: now also U3.33 (SDI)
- net OUT_AMP1: now also C35.1, R9.2, U2.8 (AINP); no longer R4.2
- net OUT_AMP2: now also C34.1, R8.2, U3.8 (AINP)
- net SCK_SPI1: now also U2.32 (SCLK)
- net SCK_SPI2: now also U3.32 (SCLK); no longer U1.21 (PB10)
- net VBUS_fuse: now also U11.3 (IN)
- net at R2.1: now also U2.34 (SDO)
- net at R3.1: now also U3.34 (SDO)
- net SCK_SPI3: now reaches U1.18 (PB0)
- net SCK_SPI3: now also U4.32 (SCLK)
- net MISO_SPI3: now reaches U1.19 (PB1)
- net MISO_SPI3: now also R4.2
- net MOSI_SPI3: now reaches U1.20 (PB2)
- net MOSI_SPI3: now also U4.33 (SDI)
- net CS_SPI2: now reaches U1.25 (PB12)
- net CS_SPI2: now also U3.31 (~{CS})
- net at R4.1: now also U4.34 (SDO)
- net CS_SPI renamed CS_SPI1
- net CS_SPI1: now also U2.31 (~{CS})
- net REFIN1 renamed REFIN
- net REFIN: now also C30.1, C6.2, C9.2, U2.4 (REFP), U3.4 (REFP), U4.4 (REFP), U9.6 (VOUT)
- net SCL_I2C1: no longer names the net of U1.43 (PB7)
- net SDA_I2C1: no longer names the net of U1.42 (PB6)
- net SDA_I2C2: no longer names the net of U1.22 (PB11)
- new net: R7.1, U5.2 (-IN), U5.6 (OUT)
- new net: R9.1, U8.2 (-IN), U8.6 (OUT)
- new net: R8.1, U7.2 (-IN), U7.6 (OUT)
- new net +AMP3: U4.7 (MXO), U5.3 (+IN)
- new net A32: U3.28 (CH0)
- new net A33: U3.27 (CH1)
- new net A34: U3.26 (CH2)
- new net A35: U3.25 (CH3)
- new net A36: U3.24 (CH4)
- new net A37: U3.23 (CH5)
- new net A38: U3.22 (CH6)
- new net A39: U3.21 (CH7)
- new net A40: U3.18 (CH8)
- new net A41: U3.17 (CH9)
- new net A42: U3.16 (CH10)
- new net A43: U3.15 (CH11)
- new net A44: U3.14 (CH12)
- new net A45: U3.13 (CH13)
- new net A46: U3.12 (CH14)
- new net A47: U3.11 (CH15)
- new net CS_SPI3: U1.21 (PB10), U4.31 (~{CS})
- new net OUT_AMP3: C32.1, R7.2, U4.8 (AINP)
- no-connect marks 57 -> 41
Other:
- added sheet Connectors (conn.kicad_sch)
- note added: "ADC3"
- note added: "REFERENCE VOLTAGE FOR ADC"
- note removed: "CONNECTOR FOR EXTERNAL ADC"
- note removed: "EXTRA I2C CONNECTOR"
- note removed: "REFERENCE VOLTAGE FOR ADC1"
- note removed: "REFERENCE VOLTAGE FOR ADC2"
- moved on the sheet: C1, C10, C11, C12, C14, C15, C16, C17, C19, C2, C20, C21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
